Commit message: Increased ball shooter shot power from 65 to 70

File: src/vrx/vrx_urdf/wamv_gazebo/urdf/components/ball_shooter.xacro (robot description, xacro)
@@ -48,5 +48,5 @@
       <!-- Adjust yaw angle (Rotate left right) -->
       <axis xyz="0 0 1"/>
-      <limit effort="1000.0" lower="${-pi/2}" upper="${pi/2}" velocity="5"/>
+      <limit effort="1000.0" lower="${-pi/2}" upper="${pi/2}" velocity="3"/>
       <origin xyz="${x} ${y} ${z}" rpy="0 0 ${yaw}"/>
       <parent link="${namespace}/base_link"/>
@@ -56,5 +56,5 @@
       <!-- Adjust pitch angle (Rotate up down)-->
       <axis xyz="0 1 0"/>
-      <limit effort="1000.0" lower="${-pi/2}" upper="0" velocity="5"/>
+      <limit effort="1000.0" lower="${-pi/2}" upper="${pi/2}" velocity="0.5"/>
       <origin xyz="-0.0204 0 0.107877" rpy="0 ${pitch} 0"/>
       <parent link="${namespace}/${name}_base_link"/>
@@ -101,5 +101,5 @@
           <pose>0.14 0 0 0 0 0</pose>
         </projectile>
-        <shot_force>65</shot_force>
+        <shot_force>70</shot_force>
         <topic>${namespace}/${shooter_namespace}${name}/fire</topic>
       </plugin>

Commit message: Added ros2_control

File: src/vrx/vrx_urdf/wamv_gazebo/urdf/components/ball_shooter.xacro (robot description, xacro)
@@ -129,4 +129,25 @@
       </plugin>
     </gazebo>
+    <!-- ros2_control -->
+    <ros2_control name="GazeboSystem" type="system">
+      <hardware>
+        <plugin>gz_ros2_control/GazeboSimSystem</plugin>
+      </hardware>
+      <joint name="wamv/ball_shooter_launcher_joint">
+        <command_interface name="position"/>
+          <param name="min">-1.57</param>
+          <param name="max">1.57</param>
+        <state_interface name="position"/>
+      </joint>
+    </ros2_control>
+    <gazebo>
+      <plugin filename="gz_ros2_control-system" name="gz_ros2_control::GazeboSimROS2ControlPlugin">
+        <parameters>$(find wamv_gazebo)/config/ball_launcher_controller.yaml</parameters>
+        <ros>
+          <namespace>/wamv</namespace>
+          <remapping>/robot_description:=/wamv/robot_description</remapping>
+        </ros>
+      </plugin>
+    </gazebo>
   </xacro:macro>
 </robot>

Commit message: Added damping and friction, increased velocity from 0.5 to 2.0 for ball_shooter_launcher_joint

File: src/vrx/vrx_urdf/wamv_gazebo/urdf/components/ball_shooter.xacro (robot description, xacro)
@@ -56,5 +56,6 @@
       <!-- Adjust pitch angle (Rotate up down)-->
       <axis xyz="0 1 0"/>
-      <limit effort="1000.0" lower="${-pi/2}" upper="${pi/2}" velocity="0.5"/>
+      <limit effort="1000.0" lower="${-pi/2}" upper="${pi/2}" velocity="2.0"/>
+      <dynamics damping="0.7" friction="0.1"/>
       <origin xyz="-0.0204 0 0.107877" rpy="0 ${pitch} 0"/>
       <parent link="${namespace}/${name}_base_link"/>

Commit message: Added damping,friction for ball_shooter_base_joint. Added ball_shooter_base_joint under <ros2_control> tag

File: src/vrx/vrx_urdf/wamv_gazebo/urdf/components/ball_shooter.xacro (robot description, xacro)
@@ -48,5 +48,6 @@
       <!-- Adjust yaw angle (Rotate left right) -->
       <axis xyz="0 0 1"/>
-      <limit effort="1000.0" lower="${-pi/2}" upper="${pi/2}" velocity="3"/>
+      <limit effort="1000.0" lower="${-pi/2}" upper="${pi/2}" velocity="3.0"/>
+      <dynamics damping="0.7" friction="0.1"/>
       <origin xyz="${x} ${y} ${z}" rpy="0 0 ${yaw}"/>
       <parent link="${namespace}/base_link"/>
@@ -141,4 +142,10 @@
         <state_interface name="position"/>
       </joint>
+      <joint name="wamv/ball_shooter_base_joint">
+        <command_interface name="position"/>
+          <param name="min">-1.57</param>
+          <param name="max">1.57</param>
+        <state_interface name="position"/>
+      </joint>
     </ros2_control>
     <gazebo>
